File: hw/sch_pcb/TFFLIP2PH.kicad_pcb (KiCad board)
At the start: 2 copper layers, 65.3 x 15.7 mm, 11 parts, among them J1 Flipper_Zero, J2 SM10B-GHS-TB, J3 SM06B-GHS-TB, J4 Angled Pinheader, J5 SM06B-GHS-TB, J6 SM07B-GHS-TB, J7 SM04B-GHS-TB, J8 SM06B-GHS-TB, J9 SM08B-GHS-TB

Commit message: Fixed #1
Other:
- board text added: "2026"
- board text added: "TFFLIP2PH-A"
Changed lines of the file:
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@@
 		(layer "Edge.Cuts")
+	)
+	(gr_text "2026"
+		(at 171.958 122.1486 0)
+		(layer "B.Cu" knockout)
+		(effects
+			(font
+				(size 1 1)
+				(thickness 0.1)
+			)
+			(justify left bottom mirror)
+		)
+	)
+	(gr_text "TFFLIP2PH-A"
+		(at 118.0338 121.6406 0)
+		(layer "F.SilkS")
+		(effects
+			(font
+				(size 1 1)
+				(thickness 0.1)
+			)
+			(justify left bottom)
+		)
 	)
 	(gr_text "Telemetry\nto Peripheral"
